File: electrical/v2/kicad/bike-generator-controller-v2/bike-generator-controller-v2.kicad_pcb (KiCad board)
At the start: 2 copper layers, 110 x 110 mm, 149 parts, among them J1 DC_GEN_IN/DIRECT DC VARIANT, J21 USB DATA TEST ONLY, J23 RESET/BOOT SERVICE, J25 VBUS TEST ONLY, J26 PROTECTED 1S, J27 USB4105-GF-A-120, J28 REMOTE LED, J3 I2C SERVICE, J31 RECEIVER OUTPUT, J32 SERVICE/NO EXT POWER, J33 103AT-2 NTC REQUIRED, J5 CONFIGURABLE GPIO, J7 SPARE POT0/50k, J8 3PH_GEN_IN (1=W 2=U 3=V), K1 TQ2-3V, Q10 AOY66923, Q11 AOY66923, Q12 AOY66923, Q13 AOY66923, Q20 AO3401A, Q21 NX6008NBKR, Q22 AO3401A, U2 ESP32-C3-MINI-1-N4X, U3 MCP4251-503E/SL, U6 TP4057-42-SOT26-R, U7 RT9080-33GJ5, U8 USBLC6-2SC6, U9 BQ25756RRVR

Commit message: chore(electrical): checkpoint controller variants, reviews and approved follow-ups
Parts:
- J27: value USB4105-GF-A-120 -> DX07S016JA1R1500; footprint Connector_USB:USB_C_Receptacle_GCT_USB4105-xx-A_16P_TopMnt_Horizontal -> Connector_USB:USB_C_Receptacle_JAE_DX07S016JA1R1500
- moved R34 73.7 mm to (50.8, 28.5)
- moved R10 70.7 mm to (47.6, 28.5), turned to 90 degrees
- moved R9 67.9 mm to (45.1, 28.5), turned to 90 degrees
- moved J5 66.3 mm to (40.0, 24.8), turned to 90 degrees
- moved R8 65.2 mm to (42.5, 28.5), turned to 90 degrees
- moved R7 62.5 mm to (40.0, 28.5), turned to 90 degrees
- moved RV1 53.9 mm to (68.2, 76.5), turned to 180 degrees
- moved J33 32.1 mm to (68.5, 69.2), turned to 0 degrees
- moved TP43 29.0 mm to (97.5, 57.1)
- moved R70 24.9 mm to (45.5, 70.0)
- moved R67 20.6 mm to (62.0, 33.5), turned to 0 degrees
- moved TP45 12.1 mm to (49.2, 46.7)
- moved C69 5.96 mm to (84.0, 51.1), turned to 180 degrees
- moved R80 4.78 mm to (82.0, 48.2)
- moved R81 4.42 mm to (85.0, 48.2)
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Routing:
- net GND: track 0.00 -> 696.3 mm, vias 0 -> 35
- net +3V3: track 0.00 -> 188.3 mm, vias 0 -> 7
- net /USB_INTERFACE/VBUS_USB: track 0.00 -> 108.8 mm, vias 0 -> 2
- net /MAIN_CONVERTER_TBD/BQ_SYS: track 0.00 -> 85.7 mm
- net /I2C_SDA: track 0.00 -> 83.6 mm, vias 0 -> 6
- net /MAIN_CONVERTER_TBD/BQ_OUT: track 0.00 -> 82.1 mm
- net /I2C_SCL: track 0.00 -> 78.2 mm, vias 0 -> 5
- net /MAIN_CONVERTER_TBD/CV_FB: track 0.00 -> 69.7 mm, vias 0 -> 1
- net /MAIN_CONVERTER_TBD/BQ_FBG: track 0.00 -> 68.2 mm, vias 0 -> 4
- net /MAIN_CONVERTER_TBD/BQ_VAC: track 0.00 -> 62.4 mm, vias 0 -> 2
- net /MAIN_CONVERTER_TBD/BQ_SW1: track 0.00 -> 58.1 mm, vias 0 -> 1
- net /MAIN_CONVERTER_TBD/BQ_SW2: track 0.00 -> 56.8 mm, vias 0 -> 1
- net /MAIN_CONVERTER_TBD/BQ_INT: track 0.00 -> 50.3 mm, vias 0 -> 3
- net /MAIN_CONVERTER_TBD/BQ_CE: track 0.00 -> 45.4 mm, vias 0 -> 3
- net /MAIN_CONVERTER_TBD/BQ_REGN: track 0.00 -> 43.0 mm, vias 0 -> 4
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