File: electrical/v2/kicad/bike-generator-controller-v2/usb_interface.kicad_sch (KiCad schematic)
At the start: 6 parts, among them J25 VBUS TEST ONLY, J27 USB4105-GF-A-120, U8 USBLC6-2SC6

Commit message: chore(electrical): checkpoint controller variants, reviews and approved follow-ups
Parts:
- J27: value USB4105-GF-A-120 -> DX07S016JA1R1500; footprint Connector_USB:USB_C_Receptacle_GCT_USB4105-xx-A_16P_TopMnt_Horizontal -> Connector_USB:USB_C_Receptacle_JAE_DX07S016JA1R1500; Design_Status PROVISIONAL USB2 - not released -> PROVISIONAL USB2 - JAE SJ121836 pin map checked; not releas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; MPN USB4105-GF-A-120 -> DX07S016JA1R1500; Manufacturer GCT -> JAE
Other:
- note added: "Provisional J27: JAE DX07S016JA1R1500 / ESD: ST USBLC6-2SC6. JAE pin map and fabrication hold: docs/USB_JAE_SELECTION_2026-10-14.md. Do not connect a valuable PC to generator-powered prototype before fault review."
- note removed: "Exact models unchanged: GCT USB4105-GF-A-120 / ST USBLC6-2SC6. Pin and package validation: electrical/components/ti-lv-power-v2/. Do not connect a valuable PC to generator-powered prototype before fault review."
Changed lines of the file:
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@@
 	(generator_version "10.0")
 	(paper "A4")
-	(text "Exact models unchanged: GCT USB4105-GF-A-120 / ST USBLC6-2SC6.\nPin and package validation: electrical/components/ti-lv-power-v2/.\nDo not connect a valuable PC to generator-powered prototype before fault review."
-		(exclude_from_sim no)
-		(at 25.4 165.1 0)
-		(effects
-			(font
-				(size 1.27 1.27)
-			)
-			(justify left top)
-		)
-	)
 	(text "USB INTERFACE - LOGIC POWER AND DATA - PROVISIONAL"
 		(exclude_from_sim no)
@@
 		)
 	)
+  (text "Provisional J27: JAE DX07S016JA1R1500 / ESD: ST USBLC6-2SC6.\nJAE pin map and fabrication hold: docs/USB_JAE_SELECTION_2026-10-14.md.\nDo not connect a valuable PC to generator-powered prototype before fault review."
+    (at 25.4 165.1 0)
+    (effects (font (size 1.27 1.27)) (justify left top))
+  )
 	(symbol
 		(lib_id "power:GND")
@@
 			)
 		)
-		(property "Value" "USB4105-GF-A-120"
+		(property "Value" "DX07S016JA1R1500"
 			(at 68.58 57.785 0)
 			(show_name no)
@@
 			)
 		)
-		(property "Footprint" "Connector_USB:USB_C_Receptacle_GCT_USB4105-xx-A_16P_TopMnt_Horizontal"
+		(property "Footprint" "Connector_USB:USB_C_Receptacle_JAE_DX07S016JA1R1500"
 			(at 68.58 77.47 0)
 			(hide yes)
@@
 			)
 		)
-		(property "Datasheet" "https://www.usb.org/sites/default/files/documents/usb_type-c.zip"
+		(property "Datasheet" "https://www.jae.com/en/connectors/series/detail/product/id=91780"
 			(at 68.58 77.47 0)
 			(hide yes)
@@
 			)
 		)
-		(property "Design_Status" "PROVISIONAL USB2 - not released"
+		(property "Design_Status" "PROVISIONAL USB2 - JAE SJ121836 pin map checked; not released"
 			(at 68.58 77.47 0)
 			(hide yes)
@@
 			)
 		)
-		(property "MPN" "USB4105-GF-A-120"
+		(property "MPN" "DX07S016JA1R1500"
 			(at 68.58 77.47 0)
 			(hide yes)
@@
 			)
 		)
-		(property "Manufacturer" "GCT"
+		(property "Manufacturer" "JAE"
 			(at 68.58 77.47 0)
 			(hide yes)
